File: hw/taiko_retrofit/taiko_retrofit.kicad_sch (KiCad schematic)
At the start: 9 parts, among them J1 Conn_01x02, J2 Conn_01x03, J3 Conn_01x04, J4 Conn_01x02, U1 RP2040-Zero

Commit message: Update PCB layout, add thanks README
Parts:
- J2: footprint Connector_JST:JST_PH_B3B-PH-K_1x03_P2.00mm_Vertical -> Connector_JST:JST_XH_B3B-XH-A_1x03_P2.50mm_Vertical
- U1: footprint 3rdparty:RP2040 Zero -> RP2040-Zero:RP2040 Zero
Changed lines of the file:
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@@
 			)
 		)
-		(property "Footprint" "Connector_JST:JST_PH_B3B-PH-K_1x03_P2.00mm_Vertical"
+		(property "Footprint" "Connector_JST:JST_XH_B3B-XH-A_1x03_P2.50mm_Vertical"
 			(at 179.07 63.5 0)
 			(effects
@@
 			)
 		)
-		(property "Footprint" "3rdparty:RP2040 Zero"
+		(property "Footprint" "RP2040-Zero:RP2040 Zero"
 			(at 125.73 74.93 0)
 			(effects
